Commit message: update urdf

File: leap_left_urdf/robot.urdf (robot description, URDF)
Before this commit: robot onshape, 17 links, 16 joints
Links:
- link fingertip: geometry collision mesh filename=package:///leap_anyskin.stl scale=0.00092 0.00092 0.00092; visual mesh filename=package:///leap_anyskin.stl scale=0.00092 0.00092 0.00092
- link fingertip_2: geometry collision mesh filename=package:///leap_anyskin.stl scale=0.00092 0.00092 0.00092; visual mesh filename=package:///leap_anyskin.stl scale=0.00092 0.00092 0.00092
- link fingertip_3: geometry collision mesh filename=package:///leap_anyskin.stl scale=0.00092 0.00092 0.00092; visual mesh filename=package:///leap_anyskin.stl scale=0.00092 0.00092 0.00092
- link thumb_fingertip: geometry collision mesh filename=package:///thumb_fingertip.stl scale=1.25 1.25 1.25; visual mesh filename=package:///thumb_fingertip.stl scale=1.25 1.25 1.25

Commit message: simulation files

File: leap_left_urdf/robot.urdf (robot description, URDF)
Before this commit: robot onshape, 17 links, 16 joints
Links:
- link fingertip: geometry collision mesh filename=package:///leap_anyskin.stl scale=0.00096 0.00092 0.00095; visual mesh filename=package:///leap_anyskin.stl scale=0.00096 0.00092 0.00095
- link fingertip_2: geometry collision mesh filename=package:///leap_anyskin.stl scale=0.00096 0.00092 0.00095; visual mesh filename=package:///leap_anyskin.stl scale=0.00096 0.00092 0.00095
- link fingertip_3: geometry collision mesh filename=package:///leap_anyskin.stl scale=0.00096 0.00092 0.00095; visual mesh filename=package:///leap_anyskin.stl scale=0.00096 0.00092 0.00095
- link thumb_dip: geometry collision mesh filename=package:///thumb_dip.stl scale=1 0.7 1; visual mesh filename=package:///thumb_dip.stl scale=1 0.7 1
- link thumb_fingertip: geometry collision mesh filename=package:///thumb_fingertip.stl scale=1.25 1.25 1.4; visual mesh filename=package:///thumb_fingertip.stl scale=1.25 1.25 1.4

Commit message: .

File: leap_left_urdf/robot.urdf (robot description, URDF)
Before this commit: robot onshape, 17 links, 16 joints
Links:
- link fingertip: geometry collision mesh filename=package:///leap_anyskin.stl scale=0.00098 0.00094 0.00097; visual mesh filename=package:///leap_anyskin.stl scale=0.00098 0.00094 0.00097
- link fingertip_2: geometry collision mesh filename=package:///leap_anyskin.stl scale=0.00098 0.00094 0.00097; visual mesh filename=package:///leap_anyskin.stl scale=0.00098 0.00094 0.00097
- link fingertip_3: geometry collision mesh filename=package:///leap_anyskin.stl scale=0.00098 0.00094 0.00097; visual mesh filename=package:///leap_anyskin.stl scale=0.00098 0.00094 0.00097
- link thumb_fingertip: geometry collision mesh filename=package:///thumb_fingertip.stl scale=1.26 1.26 1.5; visual mesh filename=package:///thumb_fingertip.stl scale=1.26 1.26 1.5
