Commit message: fixed positions

File: pb_simulation/leap_left_urdf/robot.urdf (robot description, URDF)
Before this commit: robot onshape, 17 links, 16 joints
Links:
- link fingertip: geometry collision mesh filename=package:///leap_anyskin.stl scale=0.001 0.00097 0.001; visual mesh filename=package:///leap_anyskin.stl scale=0.001 0.00097 0.001
- link fingertip_2: geometry collision mesh filename=package:///leap_anyskin.stl scale=0.001 0.00097 0.001; visual mesh filename=package:///leap_anyskin.stl scale=0.001 0.00097 0.001
- link fingertip_3: geometry collision mesh filename=package:///leap_anyskin.stl scale=0.001 0.00097 0.001; visual mesh filename=package:///leap_anyskin.stl scale=0.001 0.00097 0.001
- link pip: geometry collision mesh filename=package:///pip.stl scale=1 1 1.15; visual mesh filename=package:///pip.stl scale=1 1 1.15
- link pip_2: geometry collision mesh filename=package:///pip.stl scale=1 1 1.15; visual mesh filename=package:///pip.stl scale=1 1 1.15
- link pip_3: geometry collision mesh filename=package:///pip.stl scale=1 1 1.15; visual mesh filename=package:///pip.stl scale=1 1 1.15
